Commit message: Fix path

File: urdf/towers_of_hanoi_board.urdf.xacro (robot description, xacro)
@@ -2,7 +2,7 @@
 <robot name="edo" xmlns:xacro="http://www.ros.org/wiki/xacro">
     <!-- Import Rviz colors -->
-    <xacro:include filename="$(find edo_description)/urdf/materials.xacro" />
+    <xacro:include filename="$(find gazebo_hanoi)/urdf/materials.xacro" />
     <!--Import the edo macro -->
-    <xacro:include filename="$(find edo_games)/urdf/towers_of_hanoi_board.xacro"/>
+    <xacro:include filename="$(find gazebo_hanoi)/urdf/towers_of_hanoi_board.xacro"/>
     <xacro:arg name="board_name" default="towers_of_hanoi_board"/>
     <xacro:arg name="origin_xyz" default="0 0 0"/>

File: urdf/towers_of_hanoi_board.xacro (robot description, xacro)
@@ -24,5 +24,5 @@
                 <origin xyz="0 0 0" rpy="0 0 0"/>
                 <geometry>
-                    <mesh filename="package://edo_games/meshes/towers_of_hanoi/hanoi-board.STL"/>
+                    <mesh filename="package://gazebo_hanoi/meshes/towers_of_hanoi/hanoi-board.STL"/>
                 </geometry>
                 <material name="Brown"/>
@@ -31,5 +31,5 @@
                 <origin xyz="0 0 0" rpy="0 0 0"/>
                 <geometry>
-                    <mesh filename="package://edo_games/meshes/towers_of_hanoi/hanoi-board.STL"/>
+                    <mesh filename="package://gazebo_hanoi/meshes/towers_of_hanoi/hanoi-board.STL"/>
                 </geometry>
                 <material name="Brown"/>
