Commit message: Use boxes

File: urdf/towers_of_hanoi_token_d200.urdf (robot description, URDF)
Before this commit: robot token_d200, 1 links, 0 joints
Links:
- link token_d200_link: geometry collision box size=0.02 0.02 0.0067; visual box size=0.02 0.02 0.0067

File: urdf/towers_of_hanoi_token_d240.urdf (robot description, URDF)
Before this commit: robot token_d240, 1 links, 0 joints
Links:
- link token_d240_link: geometry collision box size=0.024 0.024 0.0067; visual box size=0.024 0.024 0.0067

File: urdf/towers_of_hanoi_token_d295.urdf (robot description, URDF)
Before this commit: robot token_d295, 1 links, 0 joints
Links:
- link token_d295_link: geometry collision box size=0.0295 0.0295 0.0067; visual box size=0.0295 0.0295 0.0067

File: urdf/towers_of_hanoi_token_d340.urdf (robot description, URDF)
Before this commit: robot token_d340, 1 links, 0 joints
Links:
- link token_d340_link: geometry collision box size=0.0340 0.0340 0.0067; visual box size=0.0340 0.0340 0.0067

File: urdf/towers_of_hanoi_token_d375.urdf (robot description, URDF)
Before this commit: robot token_d375, 1 links, 0 joints
Links:
- link token_d375_link: geometry collision box size=0.0375 0.0375 0.0067; visual box size=0.0375 0.0375 0.0067

File: urdf/towers_of_hanoi_token_d395.urdf (robot description, URDF)
Before this commit: robot token_d395, 1 links, 0 joints
Links:
- link token_d395_link: geometry collision box size=0.0395 0.0395 0.0067; visual box size=0.0395 0.0395 0.0067

File: urdf/towers_of_hanoi_token_d460.urdf (robot description, URDF)
Before this commit: robot token_d460, 1 links, 0 joints
Links:
- link token_d460_link: geometry collision box size=0.0460 0.0460 0.0067; visual box size=0.0460 0.0460 0.0067

File: urdf/towers_of_hanoi_token_d520.urdf (robot description, URDF)
Before this commit: robot token_d520, 1 links, 0 joints
Links:
- link token_d520_link: geometry collision box size=0.0520 0.0520 0.0067; visual box size=0.0520 0.0520 0.0067
